File: hardware/flute.kicad_pcb (KiCad board)
At the start: 2 copper layers, 230 x 20 mm, 47 parts, among them J1 Conn_01x02, J3 Conn_01x04, SW1 C, SW2 D, SW3 E, SW4 F, SW5 G, SW6 A, SW7 H, SW8 OCTAVE?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

Commit message: fixed power issues with flash on pcb
Parts:
- moved C4 0.25 mm to (50.1, 118.0), turned to 90 degrees
- moved C16 0.23 mm to (48.5, 118.0)
- moved BT1 0.15 mm to (46.1, 119.4)
- moved C7 0.08 mm to (52.1, 118.0)
Connections:
- C4 pad 1: +3V3 -> GND
- C4 pad 2: GND -> +3V3
- U2 pad 8: GND -> +3V3
Routing:
- net +3V3: track 53.6 -> 59.6 mm
- net GND: vias 10 -> 11
Changed lines of the file:
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@@
 	(footprint "Capacitor_SMD:C_0603_1608Metric"
 		(layer "F.Cu")
-		(at 52.07 118 -90)
+		(at 52.15 118 -90)
 		(descr "Capacitor SMD 0603 (1608 Metric), square (rectangular) end terminal, IPC-7351 nominal, (Body size source: IPC-SM-782 page 76, https://www.pcb-3d.com/wordpress/wp-content/uploads/ipc-sm-782a_amendment_1_and_2.pdf), generated with kicad-footprint-generator")
 		(tags "capacitor")
 		(property "Reference" "C7"
-			(at 2.286 0 180)
+			(at 2.286 -0.45 180)
 			(layer "F.SilkS")
 			(effects
@@
 	(footprint "Capacitor_SMD:C_0603_1608Metric"
 		(layer "F.Cu")
-		(at 50.398963 118 -90)
+		(at 50.15 118 90)
 		(descr "Capacitor SMD 0603 (1608 Metric), square (rectangular) end terminal, IPC-7351 nominal, (Body size source: IPC-SM-782 page 76, https://www.pcb-3d.com/wordpress/wp-content/uploads/ipc-sm-782a_amendment_1_and_2.pdf), generated with kicad-footprint-generator")
 		(tags "capacitor")
 		(property "Reference" "C4"
-			(at -2.176 0.058926 180)
+			(at -2.3 0.55 0)
 			(layer "F.SilkS")
 			(effects
@@
 		(attr smd)
 		(fp_line
-			(start -0.14058 0.51)
-			(end 0.14058 0.51)
+			(start -0.14058 -0.51)
+			(end 0.14058 -0.51)
 			(stroke
 				(width 0.12)
@@
 		)
 		(fp_line
-			(start -0.14058 -0.51)
-			(end 0.14058 -0.51)
+			(start -0.14058 0.51)
+			(end 0.14058 0.51)
 			(stroke
 				(width 0.12)
@@
 		)
 		(fp_line
-			(start -1.48 0.73)
-			(end -1.48 -0.73)
+			(start 1.48 -0.73)
+			(end 1.48 0.73)
 			(stroke
 				(width 0.05)
@@
 		)
 		(fp_line
-			(start 1.48 0.73)
-			(end -1.48 0.73)
+			(start -1.48 -0.73)
+			(end 1.48 -0.73)
 			(stroke
 				(width 0.05)
@@
 		)
 		(fp_line
-			(start -1.48 -0.73)
-			(end 1.48 -0.73)
+			(start 1.48 0.73)
+			(end -1.48 0.73)
 			(stroke
 				(width 0.05)
@@
 		)
 		(fp_line
-			(start 1.48 -0.73)
-			(end 1.48 0.73)
+			(start -1.48 0.73)
+			(end -1.48 -0.73)
 			(stroke
 				(width 0.05)
@@
 		)
 		(fp_line
-			(start -0.8 0.4)
-			(end -0.8 -0.4)
+			(start 0.8 -0.4)
+			(end 0.8 0.4)
 			(stroke
 				(width 0.1)
@@
 		)
 		(fp_line
-			(start 0.8 0.4)
-			(end -0.8 0.4)
+			(start -0.8 -0.4)
+			(end 0.8 -0.4)
 			(stroke
 				(width 0.1)
@@
 		)
 		(fp_line
-			(start -0.8 -0.4)
-			(end 0.8 -0.4)
+			(start 0.8 0.4)
+			(end -0.8 0.4)
 			(stroke
 				(width 0.1)
@@
 		)
 		(fp_line
-			(start 0.8 -0.4)
-			(end 0.8 0.4)
+			(start -0.8 0.4)
+			(end -0.8 -0.4)
 			(stroke
 				(width 0.1)
@@
 		)
 		(pad "1" smd roundrect
-			(at -0.775 0 270)
+			(at -0.775 0 90)
 			(size 0.9 0.95)
 			(layers "F.Cu" "F.Mask" "F.Paste")
 			(roundrect_rratio 0.25)
-			(net 5 "+3V3")
+			(net 1 "GND")
 			(pintype "passive")
 		)
 		(pad "2" smd roundrect
-			(at 0.775 0 270)
+			(at 0.775 0 90)
 			(size 0.9 0.95)
 			(layers "F.Cu" "F.Mask" "F.Paste")
 			(roundrect_rratio 0.25)
-			(net 1 "GND")
+			(net 5 "+3V3")
 			(pintype "passive")
 		)
@@
 			(layers "F.Cu" "F.Mask" "F.Paste")
 			(roundrect_rratio 0.25)
-			(net 1 "GND")
+			(net 5 "+3V3")
 			(pinfunction "VCC")
 			(pintype "power_in")
@@
 	(footprint "Capacitor_SMD:C_0603_1608Metric"
 		(layer "F.Cu")
-		(at 48.727926 118 -90)
+		(at 48.5 118 -90)
 		(descr "Capacitor SMD 0603 (1608 Metric), square (rectangular) end terminal, IPC-7351 nominal, (Body size source: IPC-SM-782 page 76, https://www.pcb-3d.com/wordpress/wp-content/uploads/ipc-sm-782a_amendment_1_and_2.pdf), generated with kicad-footprint-generator")
 		(tags "capacitor")
 		(property "Reference" "C16"
-			(at 2.286 0.227926 180)
+			(at 2.286 0.15 180)
 			(layer "F.SilkS")
 			(effects
@@
 	(footprint "Battery:BatteryHolder_MYOUNG_BS-07-A1BJ001_CR2032"
 		(layer "B.Cu")
-		(at 46.25 119.4 47)
+		(at 46.1 119.4 47)
 		(descr "CR2032 battery holder https://www.lcsc.com/datasheet/lcsc_datasheet_2203021630_MYOUNG-BS-07-A1BJ001_C2979167.pdf")
 		(tags "CR2032 BR2032 BatteryHolder Battery")
@@
 	)
 	(via
-		(at 50.477926 120.320245)
+		(at 50.5 120.4)
 		(size 1)
 		(drill 0.5)
@@
 	)
 	(via
+		(at 53.15 119.3)
+		(size 0.6)
+		(drill 0.3)
+		(layers "F.Cu" "B.Cu")
+		(free yes)
+		(net 1)
+	)
+	(via
 		(at 42.6 109.95)
 		(size 1)
@@
 	)
 	(segment
+		(start 54.145171 120.5)
+		(end 54.590926 120.054245)
+		(width 0.6)
+		(layer "F.Cu")
+		(net 5)
+	)
+	(segment
 		(start 49.038609 110.094749)
 		(end 48.891974 110.094749)
@@
 	)
 	(segment
+		(start 52.123963 120.5)
+		(end 54.145171 120.5)
+		(width 0.6)
+		(layer "F.Cu")
+		(net 5)
+	)
+	(segment
 		(start 46.05 119.35)
 		(end 46 119.3)
@@
 	)
 	(segment
+		(start 46.05 117.225)
+		(end 46.025 117.25)
+		(width 0.6)
+		(layer "F.Cu")
+		(net 5)
+	)
+	(segment
+		(start 51.174 118.249)
+		(end 50.15 117.225)
+		(width 0.6)
+		(layer "F.Cu")
+		(net 5)
+	)
+	(segment
 		(start 48.84297 110.045745)
 		(end 48.108426 110.045745)
@@
 	)
 	(segment
+		(start 51.174 119.550037)
+		(end 51.174 118.249)
+		(width 0.6)
+		(layer "F.Cu")
+		(net 5)
+	)
+	(segment
 		(start 56.168319 113.645745)
 		(end 56.644275 113.645745)
@@
 	)
 	(segment
-		(start 48.727926 117.662245)
-		(end 48.727926 117.445245)
-		(width 0.2)
-		(layer "F.Cu")
-		(net 5)
-	)
-	(segment
 		(start 47.180745 110.045745)
 		(end 47.156245 110.021245)
@@
 	)
 	(segment
-		(start 45.975 117.25)
-		(end 50.282681 117.25)
-		(width 1)
-		(layer "F.Cu")
-		(net 5)
-	)
-	(segment
-		(start 50.282681 117.25)
-		(end 50.477926 117.445245)
-		(width 1)
+		(start 52.123963 120.5)
+		(end 51.174 119.550037)
+		(width 0.6)
 		(layer "F.Cu")
 		(net 5)
@@
 		(layer "F.Cu")
 		(net 5)
+	)
+	(segment
+		(start 50.15 117.225)
+		(end 46.05 117.225)
+		(width 0.6)
+		(layer "F.Cu")
+		(net 5)
