File: hardware/raspberry.kicad_sch (KiCad schematic)
At the start: 30 parts, among them J3 Conn_01x04, U1 RP2040, U2 W25Q128JVS, Y1 Crystal_GND24

Commit message: fixed power issues with flash on pcb
Connections:
- net +3V3: now also C4.2, U2.8 (VCC); no longer C4.1
- net GND: now also C4.1; no longer C4.2, U2.8 (VCC)
Changed lines of the file:
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@@
 	(symbol
 		(lib_id "power:GND")
-		(at 248.92 82.55 90)
-		(unit 1)
-		(exclude_from_sim no)
-		(in_bom yes)
-		(on_board yes)
-		(dnp no)
-		(fields_autoplaced yes)
+		(at 246.38 72.39 0)
+		(mirror x)
+		(unit 1)
+		(exclude_from_sim no)
+		(in_bom yes)
+		(on_board yes)
+		(dnp no)
 		(property "Reference" "#PWR013"
-			(at 255.27 82.55 0)
+			(at 246.38 66.04 0)
 			(effects
 				(font
@@
 		)
 		(property "Value" "GND"
-			(at 252.73 82.5499 90)
+			(at 248.158 68.58 0)
 			(effects
 				(font
@@
 		)
 		(property "Footprint" ""
-			(at 248.92 82.55 0)
+			(at 246.38 72.39 0)
 			(effects
 				(font
@@
 		)
 		(property "Datasheet" ""
-			(at 248.92 82.55 0)
+			(at 246.38 72.39 0)
 			(effects
 				(font
@@
 		)
 		(property "Description" "Power symbol creates a global label with name \"GND\" , ground"
-			(at 248.92 82.55 0)
+			(at 246.38 72.39 0)
 			(effects
 				(font
@@
 	(symbol
 		(lib_id "power:+3V3")
-		(at 246.38 72.39 0)
-		(unit 1)
-		(exclude_from_sim no)
-		(in_bom yes)
-		(on_board yes)
-		(dnp no)
-		(fields_autoplaced yes)
+		(at 248.92 82.55 270)
+		(mirror x)
+		(unit 1)
+		(exclude_from_sim no)
+		(in_bom yes)
+		(on_board yes)
+		(dnp no)
 		(property "Reference" "#PWR012"
-			(at 246.38 76.2 0)
+			(at 245.11 82.55 0)
 			(effects
 				(font
@@
 		)
 		(property "Value" "+3V3"
-			(at 246.38 67.31 0)
+			(at 254 82.55 90)
 			(effects
 				(font
@@
 		)
 		(property "Footprint" ""
-			(at 246.38 72.39 0)
+			(at 248.92 82.55 0)
 			(effects
 				(font
@@
 		)
 		(property "Datasheet" ""
-			(at 246.38 72.39 0)
+			(at 248.92 82.55 0)
 			(effects
 				(font
@@
 		)
 		(property "Description" "Power symbol creates a global label with name \"+3V3\""
-			(at 246.38 72.39 0)
-			(effects
-				(font
+			(at 248.92 82.55 0)
+			(effects
+				(font
